File: InsuDos/_autosave-InsuDos.kicad_sch (KiCad schematic)
At the start: 95 parts, among them J1 E-paper(C097), J2 USB_B_Micro, Q1 Si1308EDL, SW1 list, SW2 enter, SW3 dose, SW4 esc, U1 USBLC6-2P6, U2 TMP102xxDRL, U3 STNS01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

Commit message: ulozenie po dlhsom case orgiginal epaper display drivre pridane
Parts:
- AE1: value Antenna_Chip -> Antenna_pcb
Changed lines of the file:
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@@
 			)
 		)
-		(property "Value" "Antenna_Chip"
+		(property "Value" "Antenna_pcb"
 			(at 46.99 94.7998 90)
 			(effects
