File: InsuDos/InsuDos.kicad_pcb (KiCad board)
At the start: 4 copper layers, 57.5 x 19.8 mm, 95 parts, among them J1 E-paper(C097), J2 USB_B_Micro, Q1 Si1308EDL, SW1 list, SW2 enter, SW3 dose, SW4 esc, U1 USBLC6-2P6, U2 TMP102xxDRL, U3 STNS01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

Commit message: added 5v usb detection
pcb not finished, drc missing, 3d models missing, project needs to be cleaned up
Parts:
- added R24: 10k, Resistor_SMD:R_0402_1005Metric, B.Cu at (66.2, 158.8)
- D1, D2, D3: value PMEG3002 -> PMEG3002
- U3: value STNS01 -> STNS01
- moved C4 0.90 mm to (52.2, 162.6), turned to -90 degrees
- moved C3 0.85 mm to (53.5, 162.6), turned to -90 degrees
Connections:
- U4 pad 30: unconnected-(U4-PE4-Pad30) -> Net-(U4-PE4)
Routing:
- net Net-(U4-PE4): track 0.00 -> 10.3 mm, vias 0 -> 2
- net /5v: track 16.4 -> 20.3 mm
- net GND: track 107.4 -> 105.1 mm, vias 193 -> 192
- net Net-(U3-ntc): track 25.7 -> 27.3 mm
- net /cen: track 31.4 -> 32.4 mm
