File: InsuDos/InsuDos.kicad_sch (KiCad schematic)
At the start: 95 parts, among them J1 E-paper(C097), J2 USB_B_Micro, Q1 Si1308EDL, SW1 list, SW2 enter, SW3 dose, SW4 esc, U1 USBLC6-2P6, U2 TMP102xxDRL, U3 STNS01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

Commit message: added 5v usb detection
pcb not finished, drc missing, 3d models missing, project needs to be cleaned up
Parts:
- added R24: 10k, Resistor_SMD:R_0402_1005Metric, symbol Device:R
Connections:
- net 5v: now also R24.1
- net at U4.30 (PE4): now also R24.2
- no-connect marks 6 -> 5
Other:
- moved on the sheet: C7, C8, Y1

Commit message: astest update
Parts:
- added R25: 470k, Resistor_SMD:R_0402_1005Metric, symbol Device:R
- R24: value 10k -> 270k
Connections:
- net GND: now also R25.1
- net at R24.2, U4.30 (PE4): now also R25.2
Other:
- moved on the sheet: R24
Changed lines of the file:
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@@
 	)
 	(junction
+		(at 115.57 107.95)
+		(diameter 0)
+		(color 0 0 0 0)
+	)
+	(junction
 		(at 34.29 52.07)
 		(diameter 0)
@@
 	(wire
 		(pts
+			(xy 105.41 107.95) (xy 106.68 107.95)
+		)
+		(stroke
+			(width 0)
+			(type default)
+		)
+	)
+	(wire
+		(pts
 			(xy 43.18 187.96) (xy 43.18 190.5)
 		)
@@
 	(wire
 		(pts
-			(xy 129.54 107.95) (xy 134.62 107.95)
+			(xy 114.3 107.95) (xy 115.57 107.95)
 		)
 		(stroke
@@
 	(wire
 		(pts
+			(xy 115.57 107.95) (xy 115.57 111.76)
+		)
+		(stroke
+			(width 0)
+			(type default)
+		)
+	)
+	(wire
+		(pts
 			(xy 177.8 105.41) (xy 191.77 105.41)
 		)
@@
 	(wire
 		(pts
-			(xy 121.92 102.87) (xy 114.3 102.87)
+			(xy 121.92 102.87) (xy 118.11 102.87)
 		)
 		(stroke
@@
 	(wire
 		(pts
+			(xy 115.57 107.95) (xy 134.62 107.95)
+		)
+		(stroke
+			(width 0)
+			(type default)
+		)
+	)
+	(wire
+		(pts
 			(xy 21.59 149.86) (xy 31.75 149.86)
 		)
@@
 	(wire
 		(pts
+			(xy 115.57 120.65) (xy 115.57 119.38)
+		)
+		(stroke
+			(width 0)
+			(type default)
+		)
+	)
+	(wire
+		(pts
 			(xy 19.05 27.94) (xy 19.05 30.48)
 		)
@@
 	)
 	(label "5v"
-		(at 121.92 107.95 180)
+		(at 105.41 107.95 180)
 		(effects
 			(font
@@
 	(symbol
 		(lib_id "Device:R")
-		(at 125.73 107.95 90)
+		(at 110.49 107.95 90)
 		(unit 1)
 		(exclude_from_sim no)
@@
 		(dnp no)
 		(property "Reference" "R24"
-			(at 128.016 107.95 90)
+			(at 112.776 107.95 90)
 			(effects
 				(font
@@
 			)
 		)
-		(property "Value" "10k"
-			(at 127.254 110.49 90)
+		(property "Value" "270k"
+			(at 112.014 110.49 90)
 			(effects
 				(font
@@
 		)
 		(property "Footprint" "Resistor_SMD:R_0402_1005Metric"
-			(at 125.73 109.728 90)
+			(at 110.49 109.728 90)
 			(effects
 				(font
@@
 		)
 		(property "Datasheet" "~"
-			(at 125.73 107.95 0)
+			(at 110.49 107.95 0)
 			(effects
 				(font
@@
 		)
 		(property "Description" "Resistor"
-			(at 125.73 107.95 0)
+			(at 110.49 107.95 0)
 			(effects
 				(font
@@
 		)
 		(property "Manufacturer" "Yageo"
-			(at 125.73 107.95 0)
+			(at 110.49 107.95 0)
 			(effects
 				(font
@@
 		)
 		(property "Mfpn" " RC0402FR-7W10KL"
-			(at 125.73 107.95 0)
+			(at 110.49 107.95 0)
 			(effects
 				(font
@@
 		)
 		(property "Price" "0.012"
-			(at 125.73 107.95 0)
+			(at 110.49 107.95 0)
 			(effects
 				(font
@@
 	)
 	(symbol
+		(lib_id "power:GND")
+		(at 115.57 120.65 0)
+		(unit 1)
+		(exclude_from_sim no)
+		(in_bom yes)
+		(on_board yes)
+		(dnp no)
+		(property "Reference" "#PWR052"
+			(at 115.57 127 0)
+			(effects
+				(font
+					(size 1.27 1.27)
+				)
+				(hide yes)
+			)
+		)
+		(property "Value" "GND"
+			(at 113.03 124.46 0)
+			(effects
+				(font
+					(size 1.27 1.27)
+				)
+				(justify left)
+			)
+		)
+		(property "Footprint" ""
+			(at 115.57 120.65 0)
+			(effects
+				(font
+					(size 1.27 1.27)
+				)
+				(hide yes)
+			)
+		)
+		(property "Datasheet" ""
+			(at 115.57 120.65 0)
+			(effects
+				(font
+					(size 1.27 1.27)
+				)
+				(hide yes)
+			)
+		)
+		(property "Description" "Power symbol creates a global label with name \"GND\" , ground"
+			(at 115.57 120.65 0)
+			(effects
+				(font
+					(size 1.27 1.27)
+				)
+				(hide yes)
+			)
+		)
+		(pin "1"
+		)
+		(instances
+			(project "InsuDos"
+				(path "/daa58ce7-4445-46d7-9757-8276efe764ff"
+					(reference "#PWR052")
+					(unit 1)
+				)
+			)
+		)
+	)
+	(symbol
 		(lib_id "Device:R")
 		(at 64.77 158.75 0)
@@
 	(symbol
 		(lib_id "power:GND")
-		(at 114.3 102.87 0)
+		(at 118.11 102.87 0)
 		(unit 1)
 		(exclude_from_sim no)
@@
 		(dnp no)
 		(property "Reference" "#PWR051"
-			(at 114.3 109.22 0)
+			(at 118.11 109.22 0)
 			(effects
 				(font
@@
 		)
 		(property "Value" "GND"
-			(at 111.76 106.68 0)
+			(at 115.57 106.68 0)
 			(effects
 				(font
@@
 		)
 		(property "Footprint" ""
-			(at 114.3 102.87 0)
+			(at 118.11 102.87 0)
 			(effects
 				(font
@@
 		)
 		(property "Datasheet" ""
-			(at 114.3 102.87 0)
+			(at 118.11 102.87 0)
 			(effects
 				(font
@@
 		)
 		(property "Description" "Power symbol creates a global label with name \"GND\" , ground"
-			(at 114.3 102.87 0)
+			(at 118.11 102.87 0)
 			(effects
 				(font
@@
 					(unit 1)
 				)
+			)
+		)
+	)
+	(symbol
+		(lib_id "Device:R")
+		(at 115.57 115.57 180)
+		(unit 1)
+		(exclude_from_sim no)
+		(in_bom yes)
+		(on_board yes)
+		(dnp no)
+		(property "Reference" "R25"
+			(at 115.57 113.284 90)
+			(effects
+				(font
+					(size 1.27 1.27)
+				)
+				(justify left)
+			)
+		)
+		(property "Value" "470k"
+			(at 113.284 113.03 90)
+			(effects
+				(font
+					(size 1.27 1.27)
+				)
+				(justify left)
+			)
+		)
+		(property "Footprint" "Resistor_SMD:R_0402_1005Metric"
+			(at 117.348 115.57 90)
+			(effects
+				(font
+					(size 1.27 1.27)
+				)
+				(hide yes)
+			)
+		)
+		(property "Datasheet" "~"
+			(at 115.57 115.57 0)
+			(effects
+				(font
+					(size 1.27 1.27)
+				)
+				(hide yes)
+			)
+		)
+		(property "Description" "Resistor"
+			(at 115.57 115.57 0)
+			(effects
+				(font
+					(size 1.27 1.27)
+				)
+				(hide yes)
+			)
+		)
+		(property "Manufacturer" "Yageo"
+			(at 115.57 115.57 0)
+			(effects
+				(font
+					(size 1.27 1.27)
+				)
+				(hide yes)
+			)
+		)
+		(property "Mfpn" " RC0402FR-13470KL"
+			(at 115.57 115.57 0)
+			(effects
+				(font
+					(size 1.27 1.27)
+				)
+				(hide yes)
+			)
+		)
+		(property "Price" "0.008"
+			(at 115.57 115.57 0)
+			(effects
+				(font
+					(size 1.27 1.27)
+				)
+				(hide yes)
+			)
+		)
+		(pin "1"
+		)
+		(pin "2"
+		)
+		(instances
+			(project "InsuDos"
+				(path "/daa58ce7-4445-46d7-9757-8276efe764ff"
+					(reference "R25")
+					(unit 1)
+				)
